Commit message: Added camera

File: ur_e_description/urdf/ur5e_with_camera.urdf (robot description, URDF)
Before this commit: robot ur5e, 11 links, 10 joints
Links:
- link ee_link: geometry collision box size=0.01 0.01 0.01

Commit message: added discrete actions but not tuned / term rewards

File: ur_e_description/urdf/ur5e_with_camera.urdf (robot description, URDF)
Before this commit: robot ur5e, 11 links, 10 joints
Links:
- link ee_link: geometry collision box size=0.15 0.1 0.1
