Commit message: added a basic link, have to fix orientation

File: ur_e_description/urdf/ur5e.urdf (robot description, URDF)
Before this commit: robot ur5e, 11 links, 10 joints
Links:
- added link camera_link; collision cylinder length=.1 radius=0.01; visual cylinder length=0.1 radius=0.01
Joints:
- added joint camera_fixed_joint: type fixed, parent wrist_2_link, child camera_link, origin xyz=0.0 -0.06 0. rpy=0.0 3.14 0

Commit message: added camera joint

File: ur_e_description/urdf/ur5e.urdf (robot description, URDF)
Before this commit: robot ur5e, 12 links, 11 joints
Links:
- link camera_link: geometry collision cylinder length=.3 radius=0.01; visual cylinder length=0.3 radius=0.01
Joints:
- joint camera_fixed_joint: origin xyz=0.0 -0.06 0. rpy=0.0 3.14 0 -> xyz=0. 0. 0.15 rpy=0.0 0 0; parent wrist_2_link -> ee_link

Commit message: Integrated RGB with discrete action code

File: ur_e_description/urdf/ur5e.urdf (robot description, URDF)
Before this commit: robot ur5e, 11 links, 10 joints
Links:
- added link camera_link; collision cylinder length=.1 radius=0.01; visual cylinder length=0.1 radius=0.01
Joints:
- added joint camera_fixed_joint: type fixed, parent wrist_2_link, child camera_link, origin xyz=0.0 -0.06 0. rpy=0.0 3.14 0
- joint world_joint: origin xyz=0.0 0.0 0.0 rpy=0.0 0.0 0.0 -> xyz=0.0 0.0 0.0 rpy=0.0 0.0 3.14

Commit message: Updated code with reward changes and tree obj file

File: ur_e_description/urdf/ur5e.urdf (robot description, URDF)
Before this commit: robot ur5e, 12 links, 11 joints
Links:
- removed link camera_link
Joints:
- removed joint camera_fixed_joint

Commit message: Fixed set_camera

File: ur_e_description/urdf/ur5e.urdf (robot description, URDF)
Before this commit: robot ur5e, 11 links, 10 joints
Joints:
- joint world_joint: origin xyz=0.0 0.0 0.0 rpy=0.0 0.0 3.14 -> xyz=0.0 0.0 0.0 rpy=0.0 0.0 0

File: ur_e_description/urdf/ur5e_with_camera.urdf (robot description, URDF)
Before this commit: robot ur5e, 11 links, 10 joints
Links:
- link ee_link: geometry collision box size=0.01 0.01 0.01
