Commit message: tree with discrete action

File: ur_e_description/urdf/tree.urdf (robot description, URDF)
Before this commit: robot ur5e, 2 links, 1 joints
Links:
- link tree: geometry collision mesh filename=../meshes/project_tree.obj scale=.1 .1 .1; visual mesh filename=../meshes/project_tree.obj scale=.1 .1 .1
Joints:
- joint tree_joint: origin xyz=-.5 0.0 -.5 rpy=0.0 0.0 1.514 -> xyz=-.7 0.0 -.5 rpy=0.0 0.0 1.514

File: ur_e_description/urdf/ur5e.urdf (robot description, URDF)
Before this commit: robot ur5e, 11 links, 10 joints
Joints:
- joint world_joint: origin xyz=0.0 0.0 0.0 rpy=0.0 0.0 0.0 -> xyz=0.0 0.0 0.0 rpy=0.0 0.0 3.14

Commit message: Solving ik error

File: ur_e_description/urdf/tree.urdf (robot description, URDF)
Before this commit: robot ur5e, 2 links, 1 joints
Links:
- link tree: geometry collision mesh filename=../meshes/tree.obj scale=.1 .1 .1; visual mesh filename=../meshes/tree.obj scale=.1 .1 .1

Commit message: Changes to simulation

File: ur_e_description/urdf/tree.urdf (robot description, URDF)
Before this commit: robot ur5e, 2 links, 1 joints
Links:
- link tree: geometry collision mesh filename=../meshes/project_tree.obj scale=.1 .1 .1; visual mesh filename=../meshes/project_tree.obj scale=.1 .1 .1
