Commit message: changes in rewards

File: ur_e_description/urdf/complex_tree.urdf (robot description, URDF)
Before this commit: robot ur5e, 2 links, 1 joints
Links:
- link tree: geometry collision mesh filename=../meshes/project_tree.obj scale=.15 .15 .15; visual mesh filename=../meshes/project_tree.obj scale=.15 .15 .15

Commit message: Changed ae weights scaling

File: ur_e_description/urdf/complex_tree.urdf (robot description, URDF)
Before this commit: robot ur5e, 2 links, 1 joints
Links:
- link tree: geometry collision mesh filename=../meshes/complex_tree.obj scale=.15 .15 .15; visual mesh filename=../meshes/complex_tree.obj scale=.15 .15 .15
